Commit message: First commit of code as used during the experiment

File: config/hand.xacro (robot description, xacro)
@@ -15,5 +15,14 @@
     </group>
     <!--GROUP STATES: Purpose: Define a named state for a particular group, in terms of joint values. This is useful to define states like 'folded arms'-->
+     <group_state name="close" group="hand">
+        <joint name="panda_finger_joint1" value="0" />
+        <joint name="panda_finger_joint2" value="0" />
+    </group_state>
+    <group_state name="open" group="hand">
+        <joint name="panda_finger_joint1" value="0.04" />
+        <joint name="panda_finger_joint2" value="0.04" />
+    </group_state>
     <!--END EFFECTOR: Purpose: Represent information about an end effector.-->
+      <end_effector name="hand" parent_link="panda_link8" group="hand" parent_group="panda_arm_hand" />
     <!--DISABLE COLLISIONS: By default it is assumed that any link of the robot could potentially come into collision with any other link in the robot. This tag disables collision checking between a specified pair of links. -->
     <disable_collisions link1="panda_hand" link2="panda_leftfinger" reason="Adjacent" />

File: config/panda_arm_hand.srdf.xacro (robot description, xacro)
@@ -27,4 +27,6 @@
     <joint name="panda_joint6" value="1.571" />
     <joint name="panda_joint7" value="0.785" />
+    <joint name="panda_finger_joint1" value="0" />
+    <joint name="panda_finger_joint2" value="0" />
   </group_state>
   <!--END EFFECTOR: Purpose: Represent information about an end effector.-->
